Commit message: enderet noen ting i setup og seletet en test launch fil

File: qube_description/urdf/qube.macro.xacro (robot description, xacro)
@@ -2,7 +2,7 @@
 <robot xmlns:xacro="http://www.ros.org/wiki/xacro">
   <!-- Define properties for dimensions -->
-  <xacro:property name="stator_size" value="0.102" />  <!-- Maintain cube form -->
-  <xacro:property name="rotor_height" value="0.008" /> <!-- Thinner disk -->
-  <xacro:property name="rotor_radius" value="0.020" /> <!-- Smaller radius -->
+  <xacro:property name="stator_size" value="0.102" />
+  <xacro:property name="rotor_height" value="0.008" />
+  <xacro:property name="rotor_radius" value="0.020" />
   <xacro:property name="angle_length" value="0.020" />
   <xacro:property name="angle_width" value="0.002" />
@@ -85,5 +85,5 @@
       <axis xyz="0 0 1"/>  <!-- Rotate around Z axis -->
     </joint>
-    <!-- Fixed joint connecting rotor_link to indicator_link -->
+    <!-- joint connecting rotor_link to indicator_link -->
     <joint name="${prefix}indicator_joint" type="fixed">
       <parent link="${prefix}rotary_link"/>

File: qube_description/urdf/qube.urdf.xacro (robot description, xacro)
@@ -3,7 +3,6 @@
     <!-- Include the Qube macro -->
     <xacro:include filename="$(find qube_description)/urdf/qube.macro.xacro" />
-    <!-- Define world link -->
     <link name="world">
-        <!-- This is an empty link that serves as the root of the robot -->
+        <!-- link that serves as the root of the robot -->
     </link>
     <!-- Call the Qube macro -->
