Commit message: Fix joint name consistency and improve Qube controllers
- Updated RViz configuration for better visualization
- Fixed motor_joint naming in controllers.yaml
- Updated PID controller to use motor_joint instead of rotary_joint
- Added proper hardware interface configuration
- Created debug launch file for testing

File: qube_bringup/urdf/controlled_qube.urdf.xacro (robot description, xacro)
@@ -1,18 +1,18 @@
 <?xml version="1.0"?>
-<robot xmlns:xacro="http://ros.org/wiki/xacro" name="controlled_qube">
-  <!-- Makroargumenter -->
+<robot xmlns:xacro="http://www.ros.org/wiki/xacro" name="controlled_qube">
+  <!-- Define arguments -->
   <xacro:arg name="baud_rate" default="115200"/>
-  <xacro:arg name="device" default="/dev/ttyUSB0"/>
+  <xacro:arg name="device" default="/dev/ttyACM0"/>
   <xacro:arg name="simulation" default="false"/>
-  <!-- Inkluder original Qube URDF -->
-  <xacro:include filename="$(find qube_description)/urdf/qube.urdf.xacro" />
-  <xacro:qube/>
-  <!-- Inkluder ROS2 Control -->
-  <xacro:include filename="$(find qube_driver)/ros2_control/qube_driver.ros2_control.xacro" />
-  <xacro:qube_driver_ros2_control
-      name="qube_driver"
-      prefix=""
-      baud_rate="$(arg baud_rate)"
-      device="$(arg device)"
-      simulation="$(arg simulation)" />
+    <!-- Include the Qube macro -->
+    <xacro:include filename="$(find qube_description)/urdf/qube.urdf.xacro" />
+    <!-- Include the ros2_control macro -->
+    <xacro:include filename="$(find qube_driver)/ros2_control/qube_driver.ros2_control.xacro" />
+    <!-- Add ros2_control to the robot -->
+    <xacro:qube_driver_ros2_control
+        name="qube_driver"
+        prefix=""
+        baud_rate="$(arg baud_rate)"
+        device="$(arg device)"
+        simulation="$(arg simulation)" />
 </robot>

File: qube_description/urdf/qube.macro.xacro (robot description, xacro)
@@ -9,5 +9,5 @@
   <xacro:property name="angle_height" value="0.002" />
   <!-- Define the qube model macro -->
-  <xacro:macro name="qube" params="prefix:=''">
+  <xacro:macro name="qube" params="prefix">
     <!-- Base link - no geometry -->
     <link name="${prefix}base_link"/>
@@ -79,5 +79,5 @@
     </joint>
     <!-- Revolute joint connecting stator_link to rotor_link -->
-    <joint name="${prefix}rotary_joint" type="continuous">
+    <joint name="${prefix}motor_joint" type="continuous">
       <parent link="${prefix}stator_link"/>
       <child link="${prefix}rotary_link"/>
